File: relay_mod.kicad_pcb (KiCad board)
At the start: 2 copper layers, 46.4 x 29.2 mm, 17 parts, among them J1 Conn_01x03, J2 Screw_Terminal_01x03, K1 SANYOU_SRD_Form_C, Q1 MMSS8050-H-TP

Commit message: Made in Costa Rica
Signed-off-by: Ricardo Mena C <rgacort12@gmail.com>
Other:
- board text added: "Hecho en Costa Rica"
Changed lines of the file:
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@@
   (general
     (thickness 1.6)
-    (drawings 18)
+    (drawings 19)
     (tracks 65)
     (zones 0)
@@
       (xy 0.6604 -0.41402) (xy 0.56134 -0.54102) (xy 0.43942 -0.64516) (xy 0.29718 -0.72136)) (layer B.SilkS) (width 0.01))
   )
+  (gr_text "Hecho en Costa Rica" (at 134.493 86.106 270) (layer B.SilkS)
+    (effects (font (size 1 1) (thickness 0.2)) (justify mirror))
+  )
   (gr_text SIGN (at 117.983 88.773 270) (layer F.SilkS)

Commit message: Adding oshwa cert
Signed-off-by: Ricardo Mena C <rgacort12@gmail.com>
Parts:
- added OSHW_Mono_0.1_Scale: CR00001, OSHWA:OSHW_Mono_0.1_Scale, B.Cu at (146.4, 88.1)
- moved ? 1.09 mm to (149.7, 88.1)
- moved REF** 0.51 mm to (149.0, 83.4)
Changed lines of the file:
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@@
-(kicad_pcb (version 20171130) (host pcbnew 5.0.2+dfsg1-1~bpo9+1)
+(kicad_pcb (version 20171130) (host pcbnew 5.0.2+dfsg1-1)
   (general
     (thickness 1.6)
@@
     (tracks 65)
     (zones 0)
-    (modules 17)
+    (modules 18)
     (nets 11)
   )
@@
   )
   (module Symbol:WEEE-Logo_4.2x6mm_SilkScreen (layer B.Cu)
-    (at 148.971 83.947 90)
+    (at 148.971 83.439 90)
     (descr "Waste Electrical and Electronic Equipment Directive")
     (tags "Logo WEEE")
@@
   )
   (module SPK_Aesthetics:OSHW-LOGO-M (layer B.Cu)
-    (at 148.844 88.773 90)
+    (at 149.733 88.138 90)
     (descr "OPEN-SOURCE HARDWARE (OSHW) LOGO - MEDIUM - SILKSCREEN")
     (tags "OPEN-SOURCE HARDWARE (OSHW) LOGO - MEDIUM - SILKSCREEN")
@@
       (xy 0.6604 -0.41402) (xy 0.56134 -0.54102) (xy 0.43942 -0.64516) (xy 0.29718 -0.72136)) (layer B.SilkS) (width 0.01))
   )
+  (module OSHWA:OSHW_Mono_0.1_Scale (layer B.Cu)
+    (at 146.431 88.138 90)
+    (fp_text reference OSHW_Mono_0.1_Scale (at 0 4.132151 90) (layer B.SilkS) hide
+      (effects (font (size 1.524 1.524) (thickness 0.3048)) (justify mirror))
+    )
+    (fp_text value CR00001 (at 0 -1.8 -90) (layer B.SilkS)
+      (effects (font (size 0.59 0.59) (thickness 0.08)) (justify mirror))
+    )
+    (fp_poly (pts (xy 0.740946 0.350373) (xy 0.871253 0.350373) (xy 0.965841 -0.451314) (xy 1.078289 0.079175)
+      (xy 1.217857 0.079175) (xy 1.331628 -0.452637) (xy 1.651994 1.084151) (xy 1.782302 1.084151)
+      (xy 1.409018 -0.637184) (xy 1.28268 -0.637184) (xy 1.148404 -0.050471) (xy 1.014789 -0.637184)
+      (xy 0.888451 -0.637184) (xy 0.740946 0.350373)) (layer B.SilkS) (width 0.00254))
+    (fp_poly (pts (xy 0.016649 0.350373) (xy 0.150925 0.350373) (xy 0.150925 -0.054439) (xy 0.516711 -0.054439)
+      (xy 0.516711 0.350373) (xy 0.650987 0.350373) (xy 0.650987 -0.637184) (xy 0.516711 -0.637184)
+      (xy 0.516711 -0.166887) (xy 0.150925 -0.166887) (xy 0.150925 -0.637184) (xy 0.016649 -0.637184)
+      (xy 0.016649 0.350373)) (layer B.SilkS) (width 0.00254))
+    (fp_poly (pts (xy -0.219492 0.316639) (xy -0.219492 0.18104) (xy -0.260135 0.204925) (xy -0.300925 0.224549)
+      (xy -0.341862 0.23991) (xy -0.382578 0.250933) (xy -0.423589 0.257548) (xy -0.464893 0.259754)
+      (xy -0.523542 0.254829) (xy -0.573372 0.240056) (xy -0.614383 0.215436) (xy -0.644883 0.182877)
+      (xy -0.663184 0.14341) (xy -0.669284 0.097035) (xy -0.660354 0.039322) (xy -0.633565 -0.002846)
+      (xy -0.602403 -0.024527) (xy -0.557424 -0.043709) (xy -0.498627 -0.060392) (xy -0.428513 -0.076267)
+      (xy -0.375967 -0.090714) (xy -0.329453 -0.108123) (xy -0.288972 -0.128496) (xy -0.254523 -0.151832)
+      (xy -0.226106 -0.178132) (xy -0.198326 -0.216001) (xy -0.178482 -0.260153) (xy -0.166576 -0.310589)
+      (xy -0.162606 -0.367309) (xy -0.166099 -0.420993) (xy -0.176577 -0.469332) (xy -0.194039 -0.512327)
+      (xy -0.218487 -0.549977) (xy -0.249919 -0.582283) (xy -0.288019 -0.608953) (xy -0.332469 -0.629696)
+      (xy -0.383269 -0.644513) (xy -0.440419 -0.653403) (xy -0.503919 -0.656366) (xy -0.550295 -0.654676)
+      (xy -0.596817 -0.649605) (xy -0.643487 -0.641153) (xy -0.690303 -0.629761) (xy -0.737267 -0.614988)
+      (xy -0.784377 -0.596835) (xy -0.784377 -0.454621) (xy -0.734621 -0.483946) (xy -0.686776 -0.507538)
+      (xy -0.640841 -0.525397) (xy -0.595347 -0.537892) (xy -0.549707 -0.545388) (xy -0.503919 -0.547887)
+      (xy -0.456129 -0.545076) (xy -0.413961 -0.536642) (xy -0.377415 -0.522586) (xy -0.346492 -0.502908)
+      (xy -0.315257 -0.468512) (xy -0.296515 -0.426179) (xy -0.290268 -0.375908) (xy -0.294604 -0.330415)
+      (xy -0.307613 -0.292711) (xy -0.329294 -0.262798) (xy -0.361265 -0.238766) (xy -0.406023 -0.218702)
+      (xy -0.46357 -0.202606) (xy -0.535008 -0.186069) (xy -0.587025 -0.172364) (xy -0.633009 -0.156119)
+      (xy -0.672961 -0.137333) (xy -0.706881 -0.116008) (xy -0.734768 -0.092142) (xy -0.76197 -0.058036)
+      (xy -0.781401 -0.018556) (xy -0.793059 0.0263) (xy -0.796945 0.076529) (xy -0.7934 0.127329)
+      (xy -0.782763 0.173896) (xy -0.765036 0.216229) (xy -0.740218 0.254329) (xy -0.708309 0.288196)
+      (xy -0.670263 0.317009) (xy -0.627559 0.339419) (xy -0.580199 0.355426) (xy -0.528181 0.365031)
+      (xy -0.471508 0.368233) (xy -0.432923 0.366762) (xy -0.393015 0.362352) (xy -0.351784 0.355004)
+      (xy -0.309157 0.345155) (xy -0.265059 0.332366) (xy -0.219492 0.316639)) (layer B.SilkS) (width 0.00254))
+    (fp_poly (pts (xy -1.105184 -0.144397) (xy -0.965617 -0.144397) (xy -0.966899 -0.206843) (xy -0.970744 -0.265196)
+      (xy -0.977152 -0.319457) (xy -0.986123 -0.369624) (xy -0.997657 -0.415699) (xy -1.011754 -0.457681)
+      (xy -1.028414 -0.49557) (xy -1.047638 -0.529366) (xy -1.077146 -0.568172) (xy -1.111432 -0.599922)
+      (xy -1.150495 -0.624616) (xy -1.194335 -0.642255) (xy -1.242952 -0.652839) (xy -1.296346 -0.656366)
+      (xy -1.349741 -0.652857) (xy -1.398358 -0.642329) (xy -1.442198 -0.624782) (xy -1.481261 -0.600216)
+      (xy -1.515546 -0.568631) (xy -1.545054 -0.530028) (xy -1.564123 -0.496366) (xy -1.580649 -0.458549)
+      (xy -1.594633 -0.416577) (xy -1.606074 -0.370451) (xy -1.614973 -0.32017) (xy -1.621329 -0.265734)
+      (xy -1.625142 -0.207143) (xy -1.626414 -0.144397) (xy -1.625142 -0.081797) (xy -1.621329 -0.02331)
+      (xy -1.614973 0.031064) (xy -1.606074 0.081325) (xy -1.594633 0.127472) (xy -1.580649 0.169505)
+      (xy -1.564123 0.207426) (xy -1.545054 0.241233) (xy -1.515362 0.280038) (xy -1.480967 0.311788)
+      (xy -1.441867 0.336482) (xy -1.398064 0.354121) (xy -1.349557 0.364704) (xy -1.296346 0.368233)
+      (xy -1.242952 0.364704) (xy -1.194335 0.354121) (xy -1.150495 0.336482) (xy -1.111432 0.311788)
+      (xy -1.077146 0.280038) (xy -1.047638 0.241233) (xy -1.028414 0.207426) (xy -1.011754 0.169505)
+      (xy -0.997657 0.127472) (xy -0.986123 0.081325) (xy -0.977152 0.031064) (xy -0.970744 -0.02331)
+      (xy -0.966899 -0.081797) (xy -0.965617 -0.144397) (xy -1.105184 -0.144397) (xy -1.106434 -0.075312)
+      (xy -1.110183 -0.013135) (xy -1.11643 0.042133) (xy -1.125176 0.090493) (xy -1.13642 0.131945)
+      (xy -1.150164 0.166488) (xy -1.17592 0.207291) (xy -1.208869 0.236436) (xy -1.249011 0.253924)
+      (xy -1.296346 0.259754) (xy -1.343434 0.253924) (xy -1.383493 0.236436) (xy -1.416525 0.207291)
+      (xy -1.442528 0.166488) (xy -1.45607 0.131945) (xy -1.467149 0.090493) (xy -1.475767 0.042133)
+      (xy -1.481922 -0.013135) (xy -1.485615 -0.075312) (xy -1.486846 -0.144397) (xy -1.485615 -0.213281)
+      (xy -1.481922 -0.275293) (xy -1.475767 -0.330433) (xy -1.467149 -0.378701) (xy -1.45607 -0.420097)
+      (xy -1.442528 -0.454621) (xy -1.416525 -0.495425) (xy -1.383493 -0.524571) (xy -1.343434 -0.542058)
+      (xy -1.296346 -0.547887) (xy -1.249011 -0.542099) (xy -1.208869 -0.524736) (xy -1.17592 -0.495797)
+      (xy -1.150164 -0.455283) (xy -1.13642 -0.42074) (xy -1.125176 -0.379289) (xy -1.11643 -0.330929)
+      (xy -1.110183 -0.27566) (xy -1.106434 -0.213483) (xy -1.105184 -0.144397)) (layer B.SilkS) (width 0.00254))
+    (fp_poly (pts (xy -2.082271 0.836724) (xy -2.082271 0.752057) (xy -2.082271 -0.999484) (xy -2.082271 -1.084151)
+      (xy -1.997604 -1.084151) (xy 1.997604 -1.084151) (xy 2.082271 -1.084151) (xy 2.082271 -0.999484)
+      (xy 2.082271 0.836724) (xy 1.916572 0.836724) (xy 1.912938 -0.914818) (xy -1.912938 -0.914818)
+      (xy -1.912938 0.667391) (xy 1.342319 0.667391) (xy 1.342319 0.836724) (xy -1.997604 0.836724)
+      (xy -2.082271 0.836724)) (layer B.SilkS) (width 0.00254))
+  )
   (gr_text "Hecho en Costa Rica" (at 134.493 86.106 270) (layer B.SilkS)
